File: hardware/thermometer-c6/thermometer-c6.kicad_sch (KiCad schematic)
At the start: 86 parts, among them J1 JST-PH-2 BAT, J2 MEAS_HDR, J3 USB-C, J4 EPD FPC24 0.5mm, J5 DEBUG, Q1 AO3401A, Q2 AO3401A, Q3 Si1308EDL, Q4 AO3401A, Q5 2N7002, SW1 RESET, SW2 BOOT, U1 ESP32-C6-MINI-1-N4, U2 RT9080-33GJ5, U3 USBLC6-2SC6, U4 MCP73831-2, U5 BMP581, Y1 FC-135 32.768kHz 12.5pF

Commit message: Redraw board schematic with real wires; add BMP585 alternate footprint
Replace the label-only rendering with authored per-zone placement and
drawn wire routes (generator/layout.py): each block now reads like a
datasheet circuit, with power symbols at rail pins and labels only for
cross-zone signals. Purely local two-pin nets are anonymous (~ prefix)
and matched by exact pin set in the netlist check instead of by name.
The collision checker gained wire-segment awareness and caught a stub
direction transform bug plus four placement conflicts during the rework;
the USBLC6 flow-through pins are now modelled honestly as two nets per
line (the KiCad symbol does not join them internally).

Add BMP585 (U6, LGA-9 3.25mm, media-resistant, LCSC-stocked) as a
populate-one alternate to the BMP581 on the same LP I2C bus with its own
local footprint drawn from BST-BMP585-DS003 - covers the BMP581 stock
gap and enables weather-exposed builds. Same 0x47 strapping; firmware
BMP58x driver handles either via chip-ID.

Co-Authored-By: Claude Fable 5 <noreply@anthropic.com>
Parts:
- added C26, C27: 100nF, Capacitor_SMD:C_0402_1005Metric, symbol Device:C
- added U6: BMP585, local:Bosch_LGA-9_3.25x3.25mm, symbol local:BMP585
- L1: value 10uH (alt 47uH SWPA4030S470MT) -> 10uH SWPA4030S
- R9: value 10M (DNP) -> 10M
- Y1: value FC-135 32.768kHz 12.5pF -> 32.768kHz FC-135
Connections:
- net +3V3: now also C26.1, C27.1, U6.3 (SDO), U6.4 (VDDIO), U6.7 (CSB), U6.8 (VDD)
- net GND: now also C26.2, C27.2, U6.5 (INT), U6.6 (VSS)
- net SCL: now also U6.1 (SCX)
- net SDA: now also U6.2 (SDX)
- net USB_D+: no longer J3.A6 (D+), J3.B6 (D+), U3.3 (I/O2)
- net USB_D-: no longer J3.A7 (D-), J3.B7 (D-), U3.1 (I/O1)
- net CHG_LED_A: no longer names the net of D1.2 (A), R4.2
- net CHG_PROG: no longer names the net of R3.1, U4.5 (PROG)
- net CHG_STAT: no longer names the net of D1.1 (K), U4.1 (STAT)
- net EPD_PUMP: no longer names the net of C16.2, D5.2 (A), D6.1 (K)
- net EPD_VCOM: no longer names the net of C25.1, J4.24 (Pin_24), TP10.1
- net EPD_VDD: no longer names the net of C21.1, J4.18 (Pin_18)
- net EPD_VGH: no longer names the net of C20.1, J4.5 (Pin_5)
- net EPD_VGL: no longer names the net of C19.1, J4.4 (Pin_4)
- net EPD_VPP: no longer names the net of C22.1, J4.19 (Pin_19)
- net EPD_VSH: no longer names the net of C23.1, J4.20 (Pin_20)
- net EPD_VSL: no longer names the net of C24.1, J4.22 (Pin_22)
- net LED_A: no longer names the net of D3.2 (A), R8.2
- net RESE_A: no longer names the net of JP2.1 (A), R14.2
- net RESE_B: no longer names the net of JP3.1 (A), R15.2
- net RESE_C: no longer names the net of JP4.1 (A), R16.2
- net USB_CC1: no longer names the net of J3.A5 (CC1), R1.1
- net USB_CC2: no longer names the net of J3.B5 (CC2), R2.1
- net VBAT_RAW: no longer names the net of J1.1 (Pin_1), J2.1 (Pin_1), JP1.1 (A)
- net VDIV_PGATE: no longer names the net of Q4.1 (G), Q5.3 (D), R18.2
- net VDIV_TOP: no longer names the net of Q4.3 (D), R20.1
- new net: J3.A6 (D+), J3.B6 (D+), U3.3 (I/O2)
- new net: J3.A7 (D-), J3.B7 (D-), U3.1 (I/O1)
- no-connect marks 13 -> 14
Other:
- moved on the sheet: C1, C10, C11, C12, C13, C14, C15, C16, C17, C18, C19, C2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
