File: hardware/thermometer-c6/thermometer-c6.kicad_sch (KiCad schematic)
At the start: 89 parts, among them J1 JST-PH-2 BAT, J2 MEAS_HDR, J3 USB-C, J4 EPD FPC24 0.5mm, J5 DEBUG, Q1 AO3401A, Q2 AO3401A, Q3 Si1308EDL, Q4 AO3401A, Q5 2N7002, SW1 RESET, SW2 BOOT, U1 ESP32-C6-MINI-1-N4, U2 RT9080-33GJ5, U3 USBLC6-2SC6, U4 MCP73831-2, U5 BMP581, U6 BMP585, Y1 32.768kHz FC-135

Commit message: Polish schematic readability: per-zone visual iteration
Fix property-text rotation on rotated instances (KiCad renders field text
at symbol+property angle and mirrors justification at effective 180);
model symbol rectangles/circles, pin-number stems and zone-title bands as
autoplacer obstacles; add far and diagonal placement candidates. Hide
test-point values (they duplicate adjacent net labels). Restructure zone
H around a single GND bus bar with staggered caps, spread the booster
pump chain, reroute the load-share gate riser out of the USB label lanes,
and drop VBAT from the debug header (GND-first pin order - a one-pin-
offset plug can no longer back-drive the LDO output; battery access
stays on J2/TP1).

Co-Authored-By: Claude Fable 5 <noreply@anthropic.com>
Parts:
- JP2: value RESE 0.47R -> 0.47R
- JP3: value RESE 2.2R -> 2.2R
- JP4: value RESE 3R -> 3R
Connections:
- net DBG_IO4: now also J5.6 (Pin_6); no longer J5.7 (Pin_7)
- net DBG_IO5: now also J5.7 (Pin_7); no longer J5.8 (Pin_8)
- net DBG_IO8: now also J5.8 (Pin_8); no longer J5.9 (Pin_9)
- net DBG_RX: now also J5.5 (Pin_5); no longer J5.6 (Pin_6)
- net DBG_TX: now also J5.4 (Pin_4); no longer J5.5 (Pin_5)
- net EN: now also J5.3 (Pin_3); no longer J5.4 (Pin_4)
- net GND: now also J5.1 (Pin_1), J5.9 (Pin_9); no longer J5.3 (Pin_3)
- net VBAT: no longer J5.1 (Pin_1)
Other:
- moved on the sheet: C14, C15, C16, C17, C18, C19, C20, C21, C22, C23, C24, C25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

Commit message: Harden board per design review; enforce clean-by-design schematic checks
Review fixes (severity order): reverse-battery P-FET on the JST input
(Q6, AO3401A - a mis-crimped pigtail no longer kills the charger), EPD
gate soft-start (R24 10k + C28 10nF, ~100us EPD_VCC ramp instead of a
hard 10uF charge-share), VBUS presence divider to GPIO4 (R22/R23, dead
at 0V without USB), DNP VBAT_ADC sampling cap (C29) and DNP VBUS TVS
(D7, SMF5.0A), BMP58x INT pins released to NC per Bosch alt config.
Charging rule documented: indoors only, 0-45C (MCP73831 has no TS pin).

Add jumper-selected boost inductor: L2 47uH beside L1 10uH, JP5/JP6 on
the switch-node side so the unselected coil idles on the DC rail -
covers the GDEH0576T81 datasheet pairing (47uH + 2.2R RESE) without
desoldering.

Generator: label-over-wire overlap is now a build error (with anchor
tolerance), zone frames auto-fit their proven content extents, and a
wire-crossing report prints any no-connection crossings - the sheet
currently has zero. Rework zones A/C/E/F/I/J accordingly; I2C pull-ups
become label islands so no riser crosses the bus runs.

Co-Authored-By: Claude Fable 5 <noreply@anthropic.com>
Parts:
- added C28, C29: 10nF, Capacitor_SMD:C_0402_1005Metric, symbol Device:C
- added D7: SMF5.0A, Diode_SMD:D_SOD-123F, symbol Device:D_TVS
- added JP5: L 10uH, Jumper:SolderJumper-2_P1.3mm_Bridged_RoundedPad1.0x1.5mm, symbol Jumper:SolderJumper_2_Bridged
- added JP6: L 47uH, Jumper:SolderJumper-2_P1.3mm_Open_RoundedPad1.0x1.5mm, symbol Jumper:SolderJumper_2_Open
- added L2: 47uH SWPA4030S, Inductor_SMD:L_Sunlord_SWPA4030S, symbol Device:L
- added Q6: AO3401A, Package_TO_SOT_SMD:SOT-23, symbol Transistor_FET:AO3401A
- added R22, R23: 100k, Resistor_SMD:R_0402_1005Metric, symbol Device:R
- added R24: 10k, Resistor_SMD:R_0402_1005Metric, symbol Device:R
Connections:
- net +3V3: now also C28.1
- net EPD_PWR_EN: now also R24.2; no longer Q2.1 (G), R12.2
- net EPD_SW: now also JP5.2 (B), JP6.2 (B); no longer L1.2
- net EPD_VCC: now also L2.1
- net GND: now also C29.2, D7.2 (A2), Q6.1 (G), R23.2; no longer U5.7 (INT), U6.5 (INT)
- net VBAT_ADC: now also C29.1
- net VBUS: now also D7.1 (A1), R22.1
- net at J2.1 (Pin_1), JP1.1 (A): now also Q6.2 (S); no longer J1.1 (Pin_1)
- net DBG_IO4 renamed VBUS_SENSE
- net VBUS_SENSE: now also R22.2, R23.1
- new net: J1.1 (Pin_1), Q6.3 (D)
- new net: C28.2, Q2.1 (G), R12.2, R24.1
- new net: JP6.1 (A), L2.2
- new net: JP5.1 (A), L1.2
- no-connect marks 14 -> 16
Other:
- moved on the sheet: D2, J2, JP1, Q3, Q5, R10, R11, R19, TP1, TP2, TP3
